File: keypad pcb/keypad pcb.sch (KiCad schematic (older format))
At the start: 18 parts, among them IC0 ATMEGA32U4-AU, IC1 usb hub, J1 usb out 1, J2 usb out 2, J3 usb power input, Y0 12 mhz, Y1 ATmega crystal

Commit message: Add keyboard switches
Parts:
- added S0: 0x0, PTS526SM15SMTR2LFS, symbol mouser:PTS526_SM15_SMTR2_LFS
- added S1: 0x1, PTS526SM15SMTR2LFS, symbol mouser:PTS526_SM15_SMTR2_LFS
- added S10: 2x0, PTS526SM15SMTR2LFS, symbol mouser:PTS526_SM15_SMTR2_LFS
- added S11: 2x1, PTS526SM15SMTR2LFS, symbol mouser:PTS526_SM15_SMTR2_LFS
- added S12: 2x2, PTS526SM15SMTR2LFS, symbol mouser:PTS526_SM15_SMTR2_LFS
- added S13: 2x3, PTS526SM15SMTR2LFS, symbol mouser:PTS526_SM15_SMTR2_LFS
- added S14: 2x4, PTS526SM15SMTR2LFS, symbol mouser:PTS526_SM15_SMTR2_LFS
- added S15: 3x0, PTS526SM15SMTR2LFS, symbol mouser:PTS526_SM15_SMTR2_LFS
- added S16: 3x1, PTS526SM15SMTR2LFS, symbol mouser:PTS526_SM15_SMTR2_LFS
- added S17: 3x2, PTS526SM15SMTR2LFS, symbol mouser:PTS526_SM15_SMTR2_LFS
- added S18: 3x3, PTS526SM15SMTR2LFS, symbol mouser:PTS526_SM15_SMTR2_LFS
- added S19: 3x4, PTS526SM15SMTR2LFS, symbol mouser:PTS526_SM15_SMTR2_LFS
- added S2: 0x2, PTS526SM15SMTR2LFS, symbol mouser:PTS526_SM15_SMTR2_LFS
- added S20: 4x0, PTS526SM15SMTR2LFS, symbol mouser:PTS526_SM15_SMTR2_LFS
- added S21: 4x1, PTS526SM15SMTR2LFS, symbol mouser:PTS526_SM15_SMTR2_LFS
- added S22: 4x2, PTS526SM15SMTR2LFS, symbol mouser:PTS526_SM15_SMTR2_LFS
- added S23: 4x3, PTS526SM15SMTR2LFS, symbol mouser:PTS526_SM15_SMTR2_LFS
- added S24: 4x4, PTS526SM15SMTR2LFS, symbol mouser:PTS526_SM15_SMTR2_LFS
- added S26: 5x0, PTS526SM15SMTR2LFS, symbol mouser:PTS526_SM15_SMTR2_LFS
- added S27: 5x1, PTS526SM15SMTR2LFS, symbol mouser:PTS526_SM15_SMTR2_LFS
- added S28: 5x2, PTS526SM15SMTR2LFS, symbol mouser:PTS526_SM15_SMTR2_LFS
- added S29: 5x3, PTS526SM15SMTR2LFS, symbol mouser:PTS526_SM15_SMTR2_LFS
- added S3: 0x3, PTS526SM15SMTR2LFS, symbol mouser:PTS526_SM15_SMTR2_LFS
- added S30: 5x4, PTS526SM15SMTR2LFS, symbol mouser:PTS526_SM15_SMTR2_LFS
- added S31: 6x0, PTS526SM15SMTR2LFS, symbol mouser:PTS526_SM15_SMTR2_LFS
- added S32: 6x1, PTS526SM15SMTR2LFS, symbol mouser:PTS526_SM15_SMTR2_LFS
- added S33: 6x2, PTS526SM15SMTR2LFS, symbol mouser:PTS526_SM15_SMTR2_LFS
- added S34: 6x3, PTS526SM15SMTR2LFS, symbol mouser:PTS526_SM15_SMTR2_LFS
- added S35: 6x4, PTS526SM15SMTR2LFS, symbol mouser:PTS526_SM15_SMTR2_LFS
- added S36: 7x0, PTS526SM15SMTR2LFS, symbol mouser:PTS526_SM15_SMTR2_LFS
- added S37: 7x1, PTS526SM15SMTR2LFS, symbol mouser:PTS526_SM15_SMTR2_LFS
- added S38: 7x2, PTS526SM15SMTR2LFS, symbol mouser:PTS526_SM15_SMTR2_LFS
- added S39: 7x3, PTS526SM15SMTR2LFS, symbol mouser:PTS526_SM15_SMTR2_LFS
- added S4: 0x4, PTS526SM15SMTR2LFS, symbol mouser:PTS526_SM15_SMTR2_LFS
- added S40: 7x4, PTS526SM15SMTR2LFS, symbol mouser:PTS526_SM15_SMTR2_LFS
- added S41: 8x0, PTS526SM15SMTR2LFS, symbol mouser:PTS526_SM15_SMTR2_LFS
- added S42: 8x1, PTS526SM15SMTR2LFS, symbol mouser:PTS526_SM15_SMTR2_LFS
- added S43: 8x2, PTS526SM15SMTR2LFS, symbol mouser:PTS526_SM15_SMTR2_LFS
- added S44: 8x3, PTS526SM15SMTR2LFS, symbol mouser:PTS526_SM15_SMTR2_LFS
- added S45: 8x4, PTS526SM15SMTR2LFS, symbol mouser:PTS526_SM15_SMTR2_LFS
- added S46: 9x0, PTS526SM15SMTR2LFS, symbol mouser:PTS526_SM15_SMTR2_LFS
- added S47: 9x1, PTS526SM15SMTR2LFS, symbol mouser:PTS526_SM15_SMTR2_LFS
- added S48: 9x2, PTS526SM15SMTR2LFS, symbol mouser:PTS526_SM15_SMTR2_LFS
- added S49: 9x3, PTS526SM15SMTR2LFS, symbol mouser:PTS526_SM15_SMTR2_LFS
- added S5: 1x0, PTS526SM15SMTR2LFS, symbol mouser:PTS526_SM15_SMTR2_LFS
- added S50: 9x4, PTS526SM15SMTR2LFS, symbol mouser:PTS526_SM15_SMTR2_LFS
- added S6: 1x1, PTS526SM15SMTR2LFS, symbol mouser:PTS526_SM15_SMTR2_LFS
- added S7: 1x2, PTS526SM15SMTR2LFS, symbol mouser:PTS526_SM15_SMTR2_LFS
- added S8: 1x3, PTS526SM15SMTR2LFS, symbol mouser:PTS526_SM15_SMTR2_LFS
- added S9: 1x4, PTS526SM15SMTR2LFS, symbol mouser:PTS526_SM15_SMTR2_LFS

Commit message: added adafruit powerboost
Parts:
- added J4: adafruit powerboost 1000c conector, 10129380908001ALF, symbol mouser:10129380-908001ALF
- added JP0: usb hub bypas D-, symbol Jumper:SolderJumper_2_Open
- added JP1: usb hub bypas D+, symbol Jumper:SolderJumper_2_Open
- added TP5: reset, symbol Connector:TestPoint
- C0: value C -> 1uF
Connections:
- net +5V: now also IC0.34 (VCC_2), IC0.44 (AVCC_2), J4.8
- net at J3.A12 (GND), J3.B12 (GND), J3.S1 (SHIELD)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: now also J4.5, J4.7
- net at J3.A9 (V-BUS), J3.B9 (V-BUS): now also J4.1
- net at IC1.15 (UP_DM), TP3.1: now also JP0.2 (B)
- net at IC1.16 (UP_DP), TP4.1: now also JP1.1 (A)
- net at IC1.8 (DM2): now also R3.1, JP0.1 (A); no longer R3.2
- net at IC1.9 (DP2): now also R4.1, JP1.2 (B); no longer R4.2
- net at IC0.13 (~RESET): now also TP5.1
- net at IC0.3 (D-): now also R3.2; no longer R3.1
- net at IC0.4 (D+): now also R4.2; no longer R4.1
- new net +BATT: J4.2
- new net enable: J4.4
- new net low: J4.6
Other:
- moved on the sheet: R3, R4
Changed lines of the file:
@@
 Connection ~ 1800 8650
 Wire Wire Line
-	5700 2400 5700 2050
+	5700 2400 5700 2200
 Wire Wire Line
 	5700 2050 5050 2050
@@
 L Device:R_Small_US R3
 U 1 1 6098AE5C
-P 4300 3150
-F 0 "R3" V 4095 3150 50  0000 C CNN
-F 1 "usb keybord" V 4186 3150 50  0000 C CNN
-F 2 "" H 4300 3150 50  0001 C CNN
-F 3 "~" H 4300 3150 50  0001 C CNN
-	1    4300 3150
-	0    1    1    0
+P 6550 3450
+F 0 "R3" V 6345 3450 50  0000 C CNN
+F 1 "usb keybord" V 6436 3450 50  0000 C CNN
+F 2 "" H 6550 3450 50  0001 C CNN
+F 3 "~" H 6550 3450 50  0001 C CNN
+	1    6550 3450
+	0    -1   -1   0
 $EndComp
 $Comp
@@
 	1400 9050 1600 9050
 Wire Wire Line
-	4200 3150 2650 3150
-Wire Wire Line
-	2650 3150 2650 1550
+	6650 3450 8200 3450
 Wire Wire Line
 	2650 1550 3250 1550
@@
 L Device:R_Small_US R4
 U 1 1 6098BF1D
-P 4300 2850
-F 0 "R4" V 4095 2850 50  0000 C CNN
-F 1 "usb keybord" V 4186 2850 50  0000 C CNN
-F 2 "" H 4300 2850 50  0001 C CNN
-F 3 "~" H 4300 2850 50  0001 C CNN
-	1    4300 2850
-	0    1    1    0
-$EndComp
-Wire Wire Line
-	4200 2850 2800 2850
-Wire Wire Line
-	2800 2850 2800 1650
+P 6600 3150
+F 0 "R4" V 6395 3150 50  0000 C CNN
+F 1 "usb keybord" V 6486 3150 50  0000 C CNN
+F 2 "" H 6600 3150 50  0001 C CNN
+F 3 "~" H 6600 3150 50  0001 C CNN
+	1    6600 3150
+	0    -1   -1   0
+$EndComp
 Wire Wire Line
 	2800 1650 3250 1650
@@
 P 9500 3300
 F 0 "C0" H 9615 3346 50  0000 L CNN
-F 1 "C" H 9615 3255 50  0000 L CNN
+F 1 "1uF" H 9615 3255 50  0000 L CNN
 F 2 "" H 9538 3150 50  0001 C CNN
 F 3 "~" H 9500 3300 50  0001 C CNN
@@
 	8200 2200 9850 2200
 Wire Wire Line
-	8200 3150 8200 2200
-Wire Wire Line
-	4400 3150 8200 3150
+	6450 3450 4450 3450
 Wire Wire Line
 	8050 2300 9850 2300
-Wire Wire Line
-	8050 2850 8050 2300
-Wire Wire Line
-	4400 2850 8050 2850
 $Comp
 L mouser:ATMEGA32U4-AU IC0
@@
 	1    0    0    -1
 $EndComp
+$Comp
+L Jumper:SolderJumper_2_Open JP1
+U 1 1 60A042C5
+P 6150 2200
+F 0 "JP1" H 6150 2405 50  0000 C CNN
+F 1 "usb hub bypas D+" H 6150 2314 50  0000 C CNN
+F 2 "" H 6150 2200 50  0001 C CNN
+F 3 "~" H 6150 2200 50  0001 C CNN
+	1    6150 2200
+	1    0    0    -1
+$EndComp
+$Comp
+L Jumper:SolderJumper_2_Open JP0
+U 1 1 60A04F60
+P 4600 2550
+F 0 "JP0" H 4600 2755 50  0000 C CNN
+F 1 "usb hub bypas D-" H 4600 2664 50  0000 C CNN
+F 2 "" H 4600 2550 50  0001 C CNN
+F 3 "~" H 4600 2550 50  0001 C CNN
+	1    4600 2550
+	1    0    0    -1
+$EndComp
+Wire Wire Line
+	2800 1650 2800 3150
+Wire Wire Line
+	2800 3150 6300 3150
+Wire Wire Line
+	2650 1550 2650 3450
+Wire Wire Line
+	8200 2200 8200 3450
+Wire Wire Line
+	6700 3150 8050 3150
+Wire Wire Line
+	5700 2200 6000 2200
+Connection ~ 5700 2200
+Wire Wire Line
+	5700 2200 5700 2050
+Wire Wire Line
+	5150 2400 5000 2400
+Wire Wire Line
+	5000 2400 5000 2550
+Wire Wire Line
+	5000 2550 4750 2550
+Connection ~ 5150 2400
+Wire Wire Line
+	4450 2550 4450 3450
+Connection ~ 4450 3450
+Wire Wire Line
+	4450 3450 2650 3450
+Wire Wire Line
+	8050 2300 8050 3150
+Wire Wire Line
+	6300 2200 6300 3150
+Connection ~ 6300 3150
+Wire Wire Line
+	6300 3150 6500 3150
+$Comp
+L power:+5V #PWR?
+U 1 1 60A3BA7E
+P 10950 900
+F 0 "#PWR?" H 10950 750 50  0001 C CNN
+F 1 "+5V" H 10965 1073 50  0000 C CNN
+F 2 "" H 10950 900 50  0001 C CNN
+F 3 "" H 10950 900 50  0001 C CNN
+	1    10950 900
+	1    0    0    -1
+$EndComp
+$Comp
+L power:+5V #PWR?
+U 1 1 60A3C8D3
+P 11950 900
+F 0 "#PWR?" H 11950 750 50  0001 C CNN
+F 1 "+5V" H 11965 1073 50  0000 C CNN
+F 2 "" H 11950 900 50  0001 C CNN
+F 3 "" H 11950 900 50  0001 C CNN
+	1    11950 900
+	1    0    0    -1
+$EndComp
+$Comp
+L mouser:10129380-908001ALF J4
+U 1 1 60A4264E
+P 2000 6800
+F 0 "J4" V 2354 6928 50  0000 L CNN
+F 1 "adafruit powerboost 1000c conector" V 2445 6928 50  0000 L CNN
+F 2 "10129380908001ALF" H 2650 6900 50  0001 L CNN
+F 3 "https://cdn.amphenol-icc.com/media/wysiwyg/files/drawing/10129380.pdf" H 2650 6800 50  0001 L CNN
+F 4 "EconoStik, Board to Board connector, Unshrouded Vertical Header, Surface Mount, Single Row, 3 Positions, 2.54 mm (0.100in) Pitch." H 2650 6700 50  0001 L CNN "Description"
+F 5 "9.85" H 2650 6600 50  0001 L CNN "Height"
+F 6 "649-1012938090801ALF" H 2650 6500 50  0001 L CNN "Mouser Part Number"
+F 7 "https://www.mouser.co.uk/ProductDetail/Amphenol-FCI/10129380-908001ALF?qs=0lQeLiL1qya5lkjRb0gX8A%3D%3D" H 2650 6400 50  0001 L CNN "Mouser Price/Stock"
+F 8 "Amphenol" H 2650 6300 50  0001 L CNN "Manufacturer_Name"
+F 9 "10129380-908001ALF" H 2650 6200 50  0001 L CNN "Manufacturer_Part_Number"
+	1    2000 6800
+	0    1    1    0
+$EndComp
+Wire Wire Line
+	1700 9050 1700 8000
+Wire Wire Line
+	1700 8000 2000 8000
+Wire Wire Line
+	2000 8000 2000 7600
+$Comp
+L power:+BATT #PWR?
+U 1 1 60A4AA45
+P 2000 6800
+F 0 "#PWR?" H 2000 6650 50  0001 C CNN
+F 1 "+BATT" H 2015 6973 50  0000 C CNN
+F 2 "" H 2000 6800 50  0001 C CNN
+F 3 "" H 2000 6800 50  0001 C CNN
+	1    2000 6800
+	1    0    0    -1
+$EndComp
+Text GLabel 1900 6500 1    50   Input ~ 0
+enable
+Wire Wire Line
+	1900 6800 1900 6500
+Wire Wire Line
+	1800 7600 1800 7800
+Wire Wire Line
+	1800 7800 1600 7800
+Wire Wire Line
+	1600 7800 1600 8650
+Connection ~ 1600 8650
+Text GLabel 1800 6450 1    50   Input ~ 0
+low
+Wire Wire Line
+	1800 6800 1800 6450
+$Comp
+L power:+5V #PWR?
+U 1 1 60A5719E
+P 1700 6800
+F 0 "#PWR?" H 1700 6650 50  0001 C CNN
+F 1 "+5V" H 1715 6973 50  0000 C CNN
+F 2 "" H 1700 6800 50  0001 C CNN
+F 3 "" H 1700 6800 50  0001 C CNN
+	1    1700 6800
+	1    0    0    -1
+$EndComp
+Wire Wire Line
+	1700 7600 1800 7600
+Connection ~ 1800 7600
+$Comp
+L Connector:TestPoint TP5
+U 1 1 60A5C3D5
+P 9350 4850
+F 0 "TP5" V 9545 4922 50  0000 C CNN
+F 1 "reset" V 9454 4922 50  0000 C CNN
+F 2 "" H 9550 4850 50  0001 C CNN
+F 3 "~" H 9550 4850 50  0001 C CNN
+	1    9350 4850
+	0    -1   -1   0
+$EndComp
+Wire Wire Line
+	11050 4800 11050 4850
+Wire Wire Line
+	11050 4850 9350 4850
 $EndSCHEMATC
